File: ethero_v2.brd (EAGLE design)
At the start: 20 parts, among them IC1 ENC28J60SP, IC2 4050N, X1 RJ45-8LCT21-B

Commit message: first draft of prototype v.2
Parts:
- removed IC2: 4050N, 40xx:DIL16
- removed X1: RJ45-8LCT21-B, con-tycoelectronics:RJ45-SHIELD1
- added BEAD: 18, resistor:0204/7
- added R10, R8: 220, resistor:0204/7
- added X2: JP011821U, con-pulse:JP
- C1, C4: value (none) -> 18pF
- C2, C5: value (none) -> 100nF
- C3: value (none) -> 10uF
- R1, R2: value (none) -> 10k
- R3, R4, R6, R7: value (none) -> 50
- R5: value 2k7 -> 2k
Connections:
- removed net INT: IC1.4, IC2.3
- removed net SO: IC1.6, IC2.5
- new net LEDA: IC1.27, R8.1
- new net LEDB: IC1.26, R10.1
- new net N$10: R8.2, X2.8
- new net N$12: R10.2, X2.10
- net DCV: no longer IC2.1
- net GND: now also X2.7, X2.9, X2.SH1, X2.SH2; no longer IC2.8
- net INT0: now also IC1.4; no longer IC2.2
- net MISO: now also IC1.6; no longer IC2.4
- net TPINM: now also X2.5; no longer X1.8
- net TPINP: now also X2.4; no longer X1.7
- net TPOUTM: now also X2.3; no longer X1.2
- net TPOUTP: now also X2.2; no longer X1.1
- net V3.3: now also BEAD.1, BEAD.2, X2.1; no longer X1.3
Routing:
- net V3.3: track 231.6 -> 0.00 mm
- net GND: track 191.5 -> 87.8 mm, vias 2 -> 0
- net INT0: track 88.7 -> 0.00 mm
- net TPOUTM: track 69.1 -> 0.00 mm
- net TPOUTP: track 64.9 -> 0.00 mm
- net SS/OC1B: track 63.4 -> 0.00 mm
- net TPINP: track 46.1 -> 0.00 mm
- net RESET: track 45.6 -> 0.00 mm, vias 2 -> 0
- net DCV: track 43.5 -> 0.00 mm, vias 2 -> 0
- net TPINM: track 42.1 -> 0.00 mm
- net MOSI/OC2: track 41.5 -> 0.00 mm
- net SCK: track 39.6 -> 0.00 mm
- net INT: track 29.1 -> 0.00 mm
- net MISO: track 25.4 -> 0.00 mm
- net OSC1: track 13.2 -> 0.00 mm
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- added copper zone on layer 16, net GND

Commit message: started routing v.2
Parts:
- added C6, C9: 47u, rcl:E3,5-8
- added IC3: LP2950Z, linear:TO92
- moved R8 53.9 mm to (29.2, 15.8), turned to 180 degrees
- moved R10 45.9 mm to (29.5, 38.2), turned to 180 degrees
- moved R5 41.4 mm to (58.3, 39.5), turned to 0 degrees
- moved BEAD 41.3 mm to (29.1, 9.60)
- moved C3 40.6 mm to (71.9, 18.0)
- moved R2 40.0 mm to (68.4, 34.4)
- moved R1 39.3 mm to (70.8, 34.5), flipped to the bottom
- moved C5 37.6 mm to (35.9, 21.8), turned to 90 degrees
- moved C2 36.5 mm to (32.9, 33.8), turned to 180 degrees
- moved R4 28.7 mm to (29.2, 22.1), turned to 270 degrees
- moved R6 28.2 mm to (33.0, 27.9), turned to 0 degrees
- moved R3 27.7 mm to (31.7, 22.0), turned to 270 degrees
- moved R7 26.9 mm to (32.9, 30.2), turned to 0 degrees
- moved C1 20.7 mm to (81.0, 25.2)
- moved Q1 20.2 mm to (78.8, 34.4)
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Connections:
- removed net N$28: J1.1
- removed net N$3: J4.2, J4.3
- new net CT: BEAD.1, C5.1, R3.2, R4.2, X2.1
- net DCV: no longer R1.1, R2.1
- net GND: now also C6.-, C9.-, IC3.2, J4.2, J4.3
- net SS/OC1B: now also J1.1; no longer J1.3
- net V3.3: now also C9.+, IC3.1, R1.1, R2.1; no longer BEAD.1, C5.1, J4.5, R3.2, R4.2, X2.1
- net VIN: now also C6.+, IC3.3
Routing:
- net GND: track 87.8 -> 232.5 mm
- net SCK: track 0.00 -> 56.4 mm
- net V3.3: track 0.00 -> 49.0 mm
- net INT0: track 0.00 -> 36.7 mm
- net SS/OC1B: track 0.00 -> 36.2 mm
- net VIN: track 0.00 -> 25.3 mm
- net CT: track 0.00 -> 22.2 mm
- net N$10: track 0.00 -> 15.7 mm
- net TPOUTP: track 0.00 -> 11.2 mm
- net TPINM: track 0.00 -> 8.14 mm
- net TPINP: track 0.00 -> 8.11 mm
- net TPOUTM: track 0.00 -> 8.10 mm
- net RBIAS: track 0.00 -> 7.42 mm
- net N$5: track 0.00 -> 6.90 mm
- net N$12: track 0.00 -> 5.26 mm
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