File: ethero_v2.sch (EAGLE design)
At the start: 20 parts, among them IC1 ENC28J60SP, IC2 4050N, X1 RJ45-8LCT21-B

Commit message: first draft of prototype v.2
Parts:
- removed IC2: 4050N, 40xx:4050N
- removed X1: RJ45-8LCT21-B, con-tycoelectronics:RJ45-8LCT21-B
- added BEAD: 18, resistor:R-EU_0204/7
- added R10, R8: 220, resistor:R-EU_0204/7
- added X2: JP011821U, con-pulse:JP011821U
- C1, C4: value (none) -> 18pF
- C2, C5: value (none) -> 100nF
- C3: value (none) -> 10uF
- R1, R2: value (none) -> 10k
- R3, R4, R6, R7: value (none) -> 50
- R5: value 2k7 -> 2k
Connections:
- removed net INT: IC1.!INT, IC2A.I
- removed net SO: IC1.SO, IC2B.I
- new net LEDA: IC1.LEDA, R8.1
- new net LEDB: IC1.LEDB, R10.1
- new net N$10: R8.2, X2.A-Y
- new net N$12: R10.2, X2.C-O_A-G
- net DCV: no longer IC2P.VDD
- net GND: now also X2.A-O_C-G, X2.C-Y, X2.SH@1, X2.SH@2; no longer IC2P.VSS
- net INT0: now also IC1.!INT; no longer IC2A.O
- net MISO: now also IC1.SO; no longer IC2B.O
- net TPINM: now also X2.RD-; no longer X1.8
- net TPINP: now also X2.RD+; no longer X1.7
- net TPOUTM: now also X2.TD-; no longer X1.2
- net TPOUTP: now also X2.TD+; no longer X1.1
- net V3.3: now also BEAD.1, BEAD.2, X2.CT; no longer X1.3

Commit message: started routing v.2
Parts:
- added C6, C9: 47u, rcl:CPOL-EUE3.5-8
- added IC3: LP2950Z, linear:LP2950Z
Connections:
- removed net N$28: J1.1
- removed net N$3: J4.2, J4.3
- new net CT: BEAD.1, C5.1, R3.2, R4.2, X2.CT
- net DCV: no longer R1.1, R2.1
- net GND: now also C6.-, C9.-, IC3.GND, J4.2, J4.3
- net SS/OC1B: now also J1.1; no longer J1.3
- net V3.3: now also C9.+, IC3.O, R1.1, R2.1; no longer BEAD.1, C5.1, J4.5, R3.2, R4.2, X2.CT
- net VIN: now also C6.+, IC3.I
