File: ethero_v3.sch (EAGLE design)
At the start: 26 parts, among them IC1 ENC28J60SP, IC3 LP2950Z, X2 JP011821U

Commit message: version 3 ready for testing
Parts:
- added R9: 10k, resistor:R-EU_0204/7
- added S1: (no value), switch-omron:10-XX
Connections:
- net DCV: now also R9.2
- net GND: now also S1.P, S1.P1
- net RESET: now also R9.1, S1.S, S1.S1
Changed lines of the file:
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@@
 <part name="GND2" library="supply1" deviceset="GND" device=""/>
 <part name="C7" library="resistor" deviceset="C-EU" device="025-025X050" value="100nF"/>
+<part name="S1" library="switch-omron" deviceset="10-XX" device=""/>
+<part name="GND10" library="supply1" deviceset="GND" device=""/>
+<part name="R9" library="resistor" deviceset="R-EU_" device="0204/7" value="10k"/>
 </parts>
 <sheets>
@@
 <instance part="GND2" gate="1" x="167.64" y="81.28"/>
 <instance part="C7" gate="G$1" x="177.8" y="81.28"/>
+<instance part="S1" gate="1" x="78.74" y="48.26"/>
+<instance part="GND10" gate="1" x="78.74" y="17.78"/>
+<instance part="R9" gate="G$1" x="78.74" y="81.28" rot="R90"/>
 </instances>
 <busses>
@@
 <wire x1="40.64" y1="12.7" x2="22.86" y2="12.7" width="0.1524" layer="91"/>
 <label x="17.78" y="12.7" size="1.778" layer="95"/>
+</segment>
+<segment>
+<pinref part="R9" gate="G$1" pin="2"/>
+<wire x1="78.74" y1="86.36" x2="78.74" y2="96.52" width="0.1524" layer="91"/>
+<label x="81.28" y="93.98" size="1.778" layer="95"/>
 </segment>
 </net>
@@
 <wire x1="177.8" y1="86.36" x2="177.8" y2="83.82" width="0.1524" layer="91"/>
 </segment>
+<segment>
+<pinref part="S1" gate="1" pin="P"/>
+<wire x1="78.74" y1="43.18" x2="78.74" y2="20.32" width="0.1524" layer="91"/>
+<pinref part="S1" gate="1" pin="P1"/>
+<wire x1="78.74" y1="43.18" x2="81.28" y2="43.18" width="0.1524" layer="91"/>
+<junction x="78.74" y="43.18"/>
+<pinref part="GND10" gate="1" pin="GND"/>
+</segment>
 </net>
 <net name="INT0" class="0">
@@
 <label x="144.78" y="78.74" size="1.778" layer="95"/>
 </segment>
-</net>
+<segment>
+<pinref part="S1" gate="1" pin="S"/>
+<wire x1="78.74" y1="53.34" x2="78.74" y2="68.58" width="0.1524" layer="91"/>
+<label x="81.28" y="73.66" size="1.778" layer="95"/>
+<pinref part="S1" gate="1" pin="S1"/>
+<wire x1="78.74" y1="68.58" x2="78.74" y2="76.2" width="0.1524" layer="91"/>
+<wire x1="78.74" y1="53.34" x2="81.28" y2="53.34" width="0.1524" layer="91"/>
+<junction x="78.74" y="53.34"/>
+<pinref part="R9" gate="G$1" pin="1"/>
+<wire x1="91.44" y1="68.58" x2="78.74" y2="68.58" width="0.1524" layer="91"/>
+<junction x="78.74" y="68.58"/>
+<label x="91.44" y="66.04" size="1.778" layer="95"/>
+</segment>
+</net>
